Commit message: CHANGES IN URDF - FOR CUSTOM ROBOT MESUREMENTS + Launch file modifications

File: src/custom_robot_description/urdf/mech/rosmaster_x3_base.urdf.xacro (robot description, xacro)
@@ -51,5 +51,5 @@
     <parent link="${prefix}base_footprint"/>
     <child link="${prefix}base_link"/>
-    <origin xyz="0 0 ${wheel_radius}" rpy="0 0 0"/>
+    <origin xyz="0 0 0.051" rpy="0 0 0"/>
   </joint>
 </xacro:macro>

File: src/custom_robot_description/urdf/robots/custom_omni.urdf.xacro (robot description, xacro)
@@ -34,8 +34,6 @@
       parent="base_link"
       frame_id="laser_frame"
-      xyz_offset="0 0 0.0825"
+      xyz_offset="0.12 0 -0.038"
       rpy_offset="0 0 0"
-      mesh_xyz_offset="0 0 0"
-      mesh_rpy_offset="${-M_PI/2} 0 0"
       topic_name="scan"/>
     <xacro:imu_sensor
@@ -43,5 +41,5 @@
       parent="base_link"
       frame_id="imu"
-      xyz_offset="0 0 0.006"
+      xyz_offset="-0.065 0.027 0.01"
       rpy_offset="0 0 0"
       update_rate="15.0"

File: src/custom_robot_description/urdf/sensors/imu.urdf.xacro (robot description, xacro)
@@ -6,5 +6,5 @@
         parent:='base_link'
         frame_id:='imu'
-        xyz_offset:='0 0 0'
+        xyz_offset:='-0.065 0.027 0.01'
         rpy_offset:='0 0 0'
         inertial_xyz_offset:='0 0 0'

File: src/custom_robot_description/urdf/sensors/lidar.urdf.xacro (robot description, xacro)
@@ -7,5 +7,5 @@
     frame_id:='laser_frame'
     mesh_file:='file://$(find custom_robot_description)/meshes/rplidar/rplidar_s2.stl'
-    xyz_offset:='0 0 0.0825'
+    xyz_offset:='0.12 0 -0.038'
     rpy_offset:='0 0 0'
     mesh_xyz_offset:='0 0 0'
@@ -16,6 +16,6 @@
     inertial_xyz_offset:='0 0 0'
     inertial_rpy_offset:='0 0 0'
-    lidar_width:=0.077
-    lidar_height:=0.0398
+    lidar_width:=0.035
+    lidar_height:=0.045
     mass:=0.185
     material_name:='rplidar_black'
@@ -40,5 +40,5 @@
     <link name="${prefix}${frame_id}">
       <visual>
-        <origin xyz="${mesh_xyz_offset}" rpy="${mesh_rpy_offset}"/>
+        <origin xyz="${xyz_offset}" rpy="${mesh_rpy_offset}"/>
         <geometry>
           <mesh filename="${mesh_file}" scale="${mesh_scale}"/>
